Commit message: gripper 추가 중 (mesh파일 인식을 못 해서 gripper만 안 보이는 상태)

File: install/ur_description/share/ur_description/urdf/ur.urdf.xacro (robot description, xacro)
@@ -18,4 +18,5 @@
    <xacro:arg name="safety_pos_margin" default="0.15"/>
    <xacro:arg name="safety_k_position" default="20"/>
+   <xacro:arg name="prefix" default=""/>
    <!--When using gazebo simulations absolute paths are necessary.-->
    <xacro:arg name="force_abs_paths" default="false" />

File: install/ur_description/share/ur_description/urdf/ur_macro.xacro (robot description, xacro)
@@ -43,5 +43,6 @@
   -->
   <xacro:include filename="$(find ur_description)/urdf/inc/ur_common.xacro" />
-  <xacro:arg name="prefix" default=""/>
+  <!-- <xacro:include filename="$(find robotiq_description)/robotiq_2f_85_gripper.urdf.xacro"/> -->
+  <xacro:include filename="$(find robotiq_description)/robotiq_2f_85_macro.urdf.xacro"/>
   <xacro:macro name="ur_robot" params="
     name
@@ -373,7 +374,13 @@
     <!-- ROS-Industrial 'tool0' frame - all-zeros tool frame -->
     <link name="${tf_prefix}tool0"/>
-    <!--gripper추가-->
-    <xacro:include filename="$(find ur_description)/urdf/robotiq_2f_85_gripper.xacro" />
-    <xacro:robotiq_2f_85_gripper parent_link="${prefix}tool0" prefix="${prefix}gripper_" />
+    <xacro:robotiq_gripper
+      name="RobotiqGripperHardwareInterface"
+      parent="${tf_prefix}tool0"
+      prefix="${prefix}gripper_"
+      use_fake_hardware="true"
+      include_ros2_control="true"
+      sim_gazebo="true">
+      <origin xyz="0 0 0" rpy="0 0 0"/>
+    </xacro:robotiq_gripper>
     <joint name="${tf_prefix}flange-tool0" type="fixed">
       <!-- default toolframe - X+ left, Y+ up, Z+ front -->
