Commit message: - moveit 사용을 위해 moveit config 파일 설정 ->ur_moveit_config/srdf/ur_macro.srdf.xacro

File: install/robotiq_description/share/robotiq_description/urdf/robotiq_2f_85_gripper.urdf.xacro (robot description, xacro)
@@ -5,5 +5,5 @@
     <xacro:arg name="com_port" default="/dev/ttyUSB0" />
     <!-- Import macros -->
-    <xacro:include filename="$(find robotiq_description)/robotiq_2f_85_macro.urdf.xacro" />
+    <xacro:include filename="$(find robotiq_description)/urdf/robotiq_2f_85_macro.urdf.xacro" />
     <link name="world" />
     <xacro:robotiq_gripper name="RobotiqGripperHardwareInterface" prefix="" parent="world" use_fake_hardware="$(arg use_fake_hardware)" com_port="$(arg com_port)">

File: install/robotiq_description/share/robotiq_description/urdf/robotiq_2f_85_macro.urdf.xacro (robot description, xacro)
@@ -20,5 +20,5 @@
         gripper_closed_position:=0.7929">
         <!-- ros2 control include -->
-        <xacro:include filename="$(find robotiq_description)/2f_85.ros2_control.xacro" />
+        <xacro:include filename="$(find robotiq_description)/urdf/2f_85.ros2_control.xacro" />
         <!-- if we are simulating or directly communicating with the gripper we need a ros2 control instance -->
         <xacro:if value="${include_ros2_control}">
@@ -41,10 +41,10 @@
             <visual>
                 <geometry>
-                    <mesh filename="model://robotiq_description/meshes/visual/2f_85/robotiq_base.dae" />
-                </geometry>
-            </visual>
-            <collision>
-                <geometry>
-                    <mesh filename="model://robotiq_description/meshes/collision/2f_85/robotiq_base.stl" />
+                    <mesh filename="package://robotiq_description/meshes/visual/2f_85/robotiq_base.dae" />
+                </geometry>
+            </visual>
+            <collision>
+                <geometry>
+                    <mesh filename="package://robotiq_description/meshes/collision/2f_85/robotiq_base.stl" />
                 </geometry>
             </collision>
@@ -58,10 +58,10 @@
             <visual>
                 <geometry>
-                    <mesh filename="model://robotiq_description/meshes/visual/2f_85/left_knuckle.dae" />
-                </geometry>
-            </visual>
-            <collision>
-                <geometry>
-                    <mesh filename="model://robotiq_description/meshes/collision/2f_85/left_knuckle.stl" />
+                    <mesh filename="package://robotiq_description/meshes/visual/2f_85/left_knuckle.dae" />
+                </geometry>
+            </visual>
+            <collision>
+                <geometry>
+                    <mesh filename="package://robotiq_description/meshes/collision/2f_85/left_knuckle.stl" />
                 </geometry>
             </collision>
@@ -75,10 +75,10 @@
             <visual>
                 <geometry>
-                    <mesh filename="model://robotiq_description/meshes/visual/2f_85/right_knuckle.dae" />
-                </geometry>
-            </visual>
-            <collision>
-                <geometry>
-                    <mesh filename="model://robotiq_description/meshes/collision/2f_85/right_knuckle.stl" />
+                    <mesh filename="package://robotiq_description/meshes/visual/2f_85/right_knuckle.dae" />
+                </geometry>
+            </visual>
+            <collision>
+                <geometry>
+                    <mesh filename="package://robotiq_description/meshes/collision/2f_85/right_knuckle.stl" />
                 </geometry>
             </collision>
@@ -92,10 +92,10 @@
             <visual>
                 <geometry>
-                    <mesh filename="model://robotiq_description/meshes/visual/2f_85/left_finger.dae" />
-                </geometry>
-            </visual>
-            <collision>
-                <geometry>
-                    <mesh filename="model://robotiq_description/meshes/collision/2f_85/left_finger.stl" />
+                    <mesh filename="package://robotiq_description/meshes/visual/2f_85/left_finger.dae" />
+                </geometry>
+            </visual>
+            <collision>
+                <geometry>
+                    <mesh filename="package://robotiq_description/meshes/collision/2f_85/left_finger.stl" />
                 </geometry>
             </collision>
@@ -109,10 +109,10 @@
             <visual>
                 <geometry>
-                    <mesh filename="model://robotiq_description/meshes/visual/2f_85/right_finger.dae" />
-                </geometry>
-            </visual>
-            <collision>
-                <geometry>
-                    <mesh filename="model://robotiq_description/meshes/collision/2f_85/right_finger.stl" />
+                    <mesh filename="package://robotiq_description/meshes/visual/2f_85/right_finger.dae" />
+                </geometry>
+            </visual>
+            <collision>
+                <geometry>
+                    <mesh filename="package://robotiq_description/meshes/collision/2f_85/right_finger.stl" />
                 </geometry>
             </collision>
@@ -126,10 +126,10 @@
             <visual>
                 <geometry>
-                    <mesh filename="model://robotiq_description/meshes/visual/2f_85/left_inner_knuckle.dae" />
-                </geometry>
-            </visual>
-            <collision>
-                <geometry>
-                    <mesh filename="model://robotiq_description/meshes/collision/2f_85/left_inner_knuckle.stl" />
+                    <mesh filename="package://robotiq_description/meshes/visual/2f_85/left_inner_knuckle.dae" />
+                </geometry>
+            </visual>
+            <collision>
+                <geometry>
+                    <mesh filename="package://robotiq_description/meshes/collision/2f_85/left_inner_knuckle.stl" />
                 </geometry>
             </collision>
@@ -143,10 +143,10 @@
             <visual>
                 <geometry>
-                    <mesh filename="model://robotiq_description/meshes/visual/2f_85/right_inner_knuckle.dae" />
-                </geometry>
-            </visual>
-            <collision>
-                <geometry>
-                    <mesh filename="model://robotiq_description/meshes/collision/2f_85/right_inner_knuckle.stl" />
+                    <mesh filename="package://robotiq_description/meshes/visual/2f_85/right_inner_knuckle.dae" />
+                </geometry>
+            </visual>
+            <collision>
+                <geometry>
+                    <mesh filename="package://robotiq_description/meshes/collision/2f_85/right_inner_knuckle.stl" />
                 </geometry>
             </collision>
@@ -160,10 +160,10 @@
             <visual>
                 <geometry>
-                    <mesh filename="model://robotiq_description/meshes/visual/2f_85/left_finger_tip.dae" />
-                </geometry>
-            </visual>
-            <collision>
-                <geometry>
-                    <mesh filename="model://robotiq_description/meshes/collision/2f_85/left_finger_tip.stl" />
+                    <mesh filename="package://robotiq_description/meshes/visual/2f_85/left_finger_tip.dae" />
+                </geometry>
+            </visual>
+            <collision>
+                <geometry>
+                    <mesh filename="package://robotiq_description/meshes/collision/2f_85/left_finger_tip.stl" />
                 </geometry>
                 <surface>
@@ -195,10 +195,10 @@
             <visual>
                 <geometry>
-                    <mesh filename="model://robotiq_description/meshes/visual/2f_85/right_finger_tip.dae" />
-                </geometry>
-            </visual>
-            <collision>
-                <geometry>
-                    <mesh filename="model://robotiq_description/meshes/collision/2f_85/right_finger_tip.stl" />
+                    <mesh filename="package://robotiq_description/meshes/visual/2f_85/right_finger_tip.dae" />
+                </geometry>
+            </visual>
+            <collision>
+                <geometry>
+                    <mesh filename="package://robotiq_description/meshes/collision/2f_85/right_finger_tip.stl" />
                 </geometry>
                 <surface>

File: install/ur_description/share/ur_description/urdf/ur_macro.xacro (robot description, xacro)
@@ -44,5 +44,5 @@
   <xacro:include filename="$(find ur_description)/urdf/inc/ur_common.xacro" />
   <!-- <xacro:include filename="$(find robotiq_description)/robotiq_2f_85_gripper.urdf.xacro"/> -->
-  <xacro:include filename="$(find robotiq_description)/robotiq_2f_85_macro.urdf.xacro"/>
+  <xacro:include filename="$(find robotiq_description)/urdf/robotiq_2f_85_macro.urdf.xacro"/>
   <xacro:macro name="ur_robot" params="
     name
